Commit message: Backup current version

File: description/robot_core.xacro (robot description, xacro)
@@ -46,4 +46,7 @@
     </xacro:inertial_box>
     </link>
+    <gazebo refercence="chassis">
+        <material >Gazebo/White</material>
+    </gazebo>
     <!-- Tạo ra một joint có tên là left_wheel_joint; joint này kết nối base_link với left_wheel -->
     <joint name="left_wheel_joint" type="continuous">
@@ -69,4 +72,7 @@
     </xacro:inertial_cylinder>
     </link>
+      <gazebo refercence="left_wheel">
+        <material >Gazebo/Blue</material>
+    </gazebo>
     <!-- Tạo ra một joint có tên là right_wheel_joint; joint này kết nối base_link với right_wheel -->
     <joint name="right_wheel_joint" type="continuous">
@@ -92,4 +98,7 @@
     </xacro:inertial_cylinder>
     </link>
+      <gazebo refercence="right_wheel">
+        <material >Gazebo/Blue</material>
+    </gazebo>
     <!-- caster_wheel -->
     <joint name="caster_wheel_joint" type="fixed">
@@ -114,3 +123,6 @@
     </xacro:inertial_sphere>
     </link>
+    <gazebo refercence="caster_wheel">
+        <material >Gazebo/Black</material>
+    </gazebo>
 </robot>
